Commit message: added tutorial link to read me

File: urdf/twr.xacro (robot description, xacro)
@@ -51,4 +51,24 @@
     </inertial>
   </link>
+  <link name="link_lazer_sensor">
+    <collision name="collision_chassis">
+      <origin rpy="0 0 0" xyz="0 0 0"/>
+      <geometry>
+        <box size="${chassisLength} ${chassisWidth} ${chassisHeight}"/>
+      </geometry>
+    </collision>
+    <visual>
+      <origin rpy="0 0 0" xyz="0 0 0"/>
+      <geometry>
+        <box size="${chassisLength} ${chassisWidth} ${chassisHeight}"/>
+      </geometry>
+      <material name="blue"/>
+    </visual>
+    <inertial>
+      <mass value="${chassisMass}"/>
+      <origin rpy="0 0 0" xyz="0 0 ${-chassisHeight/4}"/>
+      <xacro:box_inertia m="${chassisMass}" x="${chassisLength}" y="${chassisWidth}" z="${chassisHeight}"/>
+    </inertial>
+  </link>
   <xacro:aruco idA="129" idB="72" tX="1" dimA="0.2" dimB="0.8"/>
   <xacro:aruco idA="35" idB="48" tX="-1" dimA="0.2" dimB="0.8"/>

Commit message: added lazer_scanner to the bot

File: urdf/twr.xacro (robot description, xacro)
@@ -51,23 +51,23 @@
     </inertial>
   </link>
-  <link name="link_lazer_sensor">
-    <collision name="collision_chassis">
-      <origin rpy="0 0 0" xyz="0 0 0"/>
+  <joint name="joint_sensor_laser" type="fixed">
+    <origin xyz="${chassisLength/2} 0 ${-chassisHeight/4}" rpy="0 0 0"/>
+    <parent link="link_chassis"/>
+    <child link="link_sensor_laser"/>
+  </joint>
+  <link name="link_sensor_laser">
+    <visual>
+      <origin xyz="0 0 0" rpy="0 0 0" />
       <geometry>
-        <box size="${chassisLength} ${chassisWidth} ${chassisHeight}"/>
+        <cylinder radius="0.1" length="0.1"/>
+      </geometry>
+      <material name="white" />
+    </visual>
+    <collision>
+      <origin xyz="0 0 0" rpy="0 0 0"/>
+      <geometry>
+        <cylinder radius="0.05" length="0.1"/>
       </geometry>
     </collision>
-    <visual>
-      <origin rpy="0 0 0" xyz="0 0 0"/>
-      <geometry>
-        <box size="${chassisLength} ${chassisWidth} ${chassisHeight}"/>
-      </geometry>
-      <material name="blue"/>
-    </visual>
-    <inertial>
-      <mass value="${chassisMass}"/>
-      <origin rpy="0 0 0" xyz="0 0 ${-chassisHeight/4}"/>
-      <xacro:box_inertia m="${chassisMass}" x="${chassisLength}" y="${chassisWidth}" z="${chassisHeight}"/>
-    </inertial>
   </link>
   <xacro:aruco idA="129" idB="72" tX="1" dimA="0.2" dimB="0.8"/>
